Commit message: some fixes for the mesh assembly

File: nikita_description/urdf/mesh_leg.xacro (robot description, xacro)
@@ -20,9 +20,9 @@
     <link name="${prefix}_coxa_link">
       <visual>
-        <origin xyz="0 -0.0052 0" rpy="0 0 0"/>
+        <origin xyz="0 0.035 -0.01" rpy="${pi / 2.0} 0 0"/>
         <geometry><mesh filename="package://nikita_description/meshes/assembly_coxa.stl" scale="${mesh_scale}"/></geometry>
         <material name="orange"/>
       </visual>
-      <collision><origin xyz="0 ${coxa_length / 2.0} 0" rpy="${-pi / 2.0} 0 0"/><geometry><box size="0.030 0.050 0.045"/></geometry></collision>
+      <collision><origin xyz="0 ${coxa_length / 2.0} 0" rpy="${pi / 2.0} 0 0"/><geometry><box size="0.030 0.050 0.045"/></geometry></collision>
       <inertial><origin xyz="0 ${coxa_length / 2.0} 0"/><mass value="0.12"/><inertia ixx="3.0e-05" ixy="0" ixz="0" iyy="3.0e-05" iyz="0" izz="3.0e-05"/></inertial>
     </link>
@@ -35,5 +35,5 @@
     <link name="${prefix}_femur_link">
       <visual>
-        <origin xyz="0 0 0" rpy="${-pi / 2.0} 0 0"/>
+        <origin xyz="0.015 0.043 0" rpy="${-pi / 2.0} ${-pi / 2.0} ${-pi}"/>
         <geometry><mesh filename="package://nikita_description/meshes/assembly_femur.stl" scale="${mesh_scale}"/></geometry>
         <material name="dark_blue"/>
@@ -50,5 +50,5 @@
     <link name="${prefix}_tibia_link">
       <visual>
-        <origin xyz="0 0 0" rpy="${-pi / 2.0} 0 0"/>
+        <origin xyz="0 0.04 0" rpy="${-pi / 2.0} 0 0"/>
         <geometry><mesh filename="package://nikita_description/meshes/assembly_tibia.stl" scale="${mesh_scale}"/></geometry>
         <material name="light_blue"/>

Commit message: further improvement of the mesh assignment

File: nikita_description/urdf/mesh_leg.xacro (robot description, xacro)
@@ -29,5 +29,5 @@
     <joint name="${prefix}_femur_joint" type="revolute">
       <parent link="${prefix}_coxa_link"/><child link="${prefix}_femur_link"/>
-      <origin xyz="0 ${coxa_length} 0" rpy="0 0 0"/><axis xyz="1 0 0"/>
+      <origin xyz="0 ${coxa_length} 0" rpy="${30 * pi / 180} 0 0"/><axis xyz="1 0 0"/>
       <limit lower="${-30 * pi / 180}" upper="${90 * pi / 180}" effort="3.0" velocity="6.0"/>
       <dynamics damping="0.1" friction="0.05"/>
@@ -35,5 +35,5 @@
     <link name="${prefix}_femur_link">
       <visual>
-        <origin xyz="0.015 0.043 0" rpy="${-pi / 2.0} ${-pi / 2.0} ${-pi}"/>
+        <origin xyz="0.015 0.043 0" rpy="${-90 * pi / 180} ${-90 * pi / 180} ${180 * pi / 180}"/>
         <geometry><mesh filename="package://nikita_description/meshes/assembly_femur.stl" scale="${mesh_scale}"/></geometry>
         <material name="dark_blue"/>
@@ -44,5 +44,5 @@
     <joint name="${prefix}_tibia_joint" type="revolute">
       <parent link="${prefix}_femur_link"/><child link="${prefix}_tibia_link"/>
-      <origin xyz="0 ${femur_length} 0" rpy="${-pi / 2.0} 0 0"/><axis xyz="1 0 0"/>
+      <origin xyz="0 ${femur_length} 0" rpy="${-120 * pi / 180} 0 0"/><axis xyz="1 0 0"/>
       <limit lower="${-90 * pi / 180}" upper="${90 * pi / 180}" effort="3.0" velocity="6.0"/>
       <dynamics damping="0.1" friction="0.05"/>
@@ -50,5 +50,5 @@
     <link name="${prefix}_tibia_link">
       <visual>
-        <origin xyz="0 0.04 0" rpy="${-pi / 2.0} 0 0"/>
+        <origin xyz="-0.015 0.04 0" rpy="${-90 * pi / 180} ${90 * pi / 180} ${180 * pi / 180}"/>
         <geometry><mesh filename="package://nikita_description/meshes/assembly_tibia.stl" scale="${mesh_scale}"/></geometry>
         <material name="light_blue"/>
